File: board/nano-m7.kicad_pcb (KiCad board)
At the start: 2 copper layers, 95 x 70 mm, 64 parts, among them J1 Z-FORCE, J10 UI PANEL, J11 HDMI POWER, J12 RASPI, J2 Z-STEPPER, J3 Z-STOP LOW, J4 LAMP NTC, J5 LAMP PWM, J6 LAMP FAN, J7 LAMP FAN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

Commit message: 1.1
Parts:
- removed the C10 at (96.5, 51.6)
- removed the C11 at (105.5, 54.6)
- removed C14: 100u/16V, Capacitor_SMD:CP_Elec_6.3x5.4
- removed L2: 6.8uH, Drake:CKCS6028
- removed R12, R15: 100k, Resistor_SMD:R_0805_2012Metric_Pad1.20x1.40mm_HandSolder
- removed R13: 30k 1%, Resistor_SMD:R_0805_2012Metric_Pad1.20x1.40mm_HandSolder
- removed R14: 6.65k 1%, Resistor_SMD:R_0805_2012Metric_Pad1.20x1.40mm_HandSolder
- removed R16: 30.9k 1%, Resistor_SMD:R_0805_2012Metric_Pad1.20x1.40mm_HandSolder
- removed R17: 4.22k 1%, Resistor_SMD:R_0805_2012Metric_Pad1.20x1.40mm_HandSolder
- added C6: 100u/35V, Capacitor_SMD:CP_Elec_6.3x5.8, F.Cu at (88.0, 72.5)
- added C7: 100n, Capacitor_SMD:C_0805_2012Metric, F.Cu at (94.0, 72.5)
- added D1: SS24, Diode_SMD:D_SMA_Handsoldering, F.Cu at (101.0, 75.5)
- C1, C2: value 22p -> 18p
- C11: renamed from C8; footprint Capacitor_SMD:C_0805_2012Metric_Pad1.18x1.45mm_HandSolder -> Capacitor_SMD:C_0805_2012Metric
- C12: value 100u/35V -> 10u; footprint Capacitor_SMD:CP_Elec_6.3x5.8 -> Capacitor_SMD:C_0805_2012Metric
- C13: value 100n -> 10u; footprint Capacitor_SMD:C_0805_2012Metric_Pad1.18x1.45mm_HandSolder -> Capacitor_SMD:C_0805_2012Metric
- C9: value 100u/35V -> 100u/16V
- J3: footprint Connector_JST:JST_XH_B2B-XH-A_1x02_P2.50mm_Vertical -> Connector_JST:JST_XH_B3B-XH-A_1x03_P2.50mm_Vertical
- L1: value 6.8uH -> 47uH/2A; footprint Drake:CKCS6028 -> Inductor_SMD:L_Sunlord_MWSA0604S
- R1, R10, R11, R2, R5, R6, R7, R9: footprint Resistor_SMD:R_0805_2012Metric_Pad1.20x1.40mm_HandSolder -> Resistor_SMD:R_0805_2012Metric
- R3: value 270R -> 330R
- R4, R8: value 1k -> 1k5; footprint Resistor_SMD:R_0805_2012Metric_Pad1.20x1.40mm_HandSolder -> Resistor_SMD:R_0805_2012Metric
- U2: value FR8205 -> XL1509-5.0; footprint Package_TO_SOT_SMD:SOT-23-6 -> Package_SO:SOIC-8_3.9x4.9mm_P1.27mm
- U3: value FR8205 -> LM1117MP-3.3; footprint Package_TO_SOT_SMD:SOT-23-6 -> Package_TO_SOT_SMD:SOT-223-3_TabPin2
- Y1: value 12MHz -> 16MHz
- moved C13 19.2 mm to (90.0, 50.6), turned to 90 degrees
- moved C12 17.0 mm to (90.0, 54.8)
- moved U2 16.3 mm to (90.0, 63.5)
- moved C9 14.7 mm to (101.0, 60.5), turned to 180 degrees
- moved U3 14.2 mm to (98.0, 51.5), turned to 0 degrees
- moved L1 13.2 mm to (101.0, 69.0)
- moved J3 3.05 mm to (146.0, 98.5)
- moved C3 2.97 mm to (128.5, 75.6)
- moved C4 2.97 mm to (126.5, 75.6)
- renumbered C7 to C10, C6 to C8, D1 to D2
Connections:
- A1 pad 2: unconnected-(A1-~{FLT}-Pad2) -> /~{ZS_FAULT}
- A1 pad 9: unconnected-(A1-~{EN}-Pad9) -> /~{ZS_EN}
- C12 pad 1: +24V -> +5V
- C13 pad 1: Net-(U3-BST) -> +3V3
- C13 pad 2: Net-(U3-LX) -> GND
- C9 pad 1: +24V -> +5V
- J3 pad 1: /Z_STOP_LOW -> +5V
- L1 pad 1: Net-(U2-LX) -> Net-(D1-K)
- L1 pad 2: +3V3 -> +5V
- U1 pad 21: unconnected-(U1-PA11-Pad21) -> /~{ZS_EN}
- U1 pad 22: unconnected-(U1-PA12-Pad22) -> /~{ZS_FAULT}
- U2 pad 1: Net-(U2-BST) -> +24V
- U2 pad 2: GND -> Net-(D1-K)
- U2 pad 3: Net-(U2-FB) -> +5V
- U2 pad 4: Net-(U2-SHDN) -> GND
- U2 pad 5: +24V -> GND
- U2 pad 6: Net-(U2-LX) -> GND
- U3 pad 1: Net-(U3-BST) -> GND
- U3 pad 2: GND -> +3V3
- U3 pad 3: Net-(U3-FB) -> +5V
Routing:
- net /~{ZS_FAULT}: track 0.00 -> 36.8 mm, vias 0 -> 4
- net +5V: track 151.0 -> 185.9 mm
- net /~{ZS_EN}: track 0.00 -> 33.1 mm, vias 0 -> 2
- net GND: track 52.8 -> 30.1 mm, vias 29 -> 82
- net +24V: track 175.5 -> 153.4 mm
- net Net-(D1-K): track 0.00 -> 15.7 mm
- net Net-(U3-FB): track 9.67 -> 0.00 mm
- net Net-(U2-FB): track 9.67 -> 0.00 mm
- net Net-(U3-LX): track 7.81 -> 0.00 mm
- net Net-(U2-LX): track 7.81 -> 0.00 mm
- net +3V3: track 192.1 -> 197.7 mm
- net /~{RST}: track 62.0 -> 57.7 mm
- net /ZS_STEP: track 18.5 -> 21.4 mm
- net Net-(U2-SHDN): track 2.88 -> 0.00 mm
- net Net-(U3-SHDN): track 2.88 -> 0.00 mm
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- added copper zone on F.Cu, net +24V
Other:
- board text added: "v1.1 drake.cz"
- board text removed: "v1.0 drake.cz"
