File: board/p-mos-switch.kicad_sch (KiCad schematic)
At the start: 6 parts, among them Q1 MMBT3904, Q2 Q_PMOS_GDS

Commit message: WIP
Parts:
- R4: value 1k -> 1k5
Changed lines of the file:
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@@
 			)
 		)
-		(property "Value" "1k"
+		(property "Value" "1k5"
 			(at 121.92 68.58 90)
 			(effects

Commit message: 1.1
Parts:
- R4, R5, R6, R7: footprint Resistor_SMD:R_0805_2012Metric_Pad1.20x1.40mm_HandSolder -> Resistor_SMD:R_0805_2012Metric
Changed lines of the file:
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@@
 			)
 		)
-		(property "Footprint" "Resistor_SMD:R_0805_2012Metric_Pad1.20x1.40mm_HandSolder"
+		(property "Footprint" "Resistor_SMD:R_0805_2012Metric"
 			(at 131.318 71.12 90)
 			(effects
@@
 			)
 		)
-		(property "Footprint" "Resistor_SMD:R_0805_2012Metric_Pad1.20x1.40mm_HandSolder"
+		(property "Footprint" "Resistor_SMD:R_0805_2012Metric"
 			(at 133.35 49.022 90)
 			(effects
@@
 		(dnp no)
 		(fields_autoplaced yes)
-		(property "Reference" "#PWR029"
+		(property "Reference" "#PWR033"
 			(at 140.97 83.82 0)
 			(effects
@@
 		)
 		(instances
-			(project ""
-				(path "/657b92bb-29fd-4612-8c57-4a7da3c6d68f/a0ec00c8-1016-421a-a89c-2f1904f8a9f7"
-					(reference "#PWR029")
-					(unit 1)
-				)
-				(path "/657b92bb-29fd-4612-8c57-4a7da3c6d68f/f2ca9a7d-fea9-4a68-835b-845e026c6569"
-					(reference "#PWR031")
+			(project "nano-m7"
+				(path "/657b92bb-29fd-4612-8c57-4a7da3c6d68f/a0ec00c8-1016-421a-a89c-2f1904f8a9f7"
+					(reference "#PWR033")
+					(unit 1)
+				)
+				(path "/657b92bb-29fd-4612-8c57-4a7da3c6d68f/f2ca9a7d-fea9-4a68-835b-845e026c6569"
+					(reference "#PWR035")
 					(unit 1)
 				)
@@
 		)
 		(instances
-			(project ""
+			(project "nano-m7"
 				(path "/657b92bb-29fd-4612-8c57-4a7da3c6d68f/a0ec00c8-1016-421a-a89c-2f1904f8a9f7"
 					(reference "Q1")
@@
 			)
 		)
-		(property "Footprint" "Resistor_SMD:R_0805_2012Metric_Pad1.20x1.40mm_HandSolder"
+		(property "Footprint" "Resistor_SMD:R_0805_2012Metric"
 			(at 121.92 64.262 90)
 			(effects
@@
 		)
 		(instances
-			(project ""
+			(project "nano-m7"
 				(path "/657b92bb-29fd-4612-8c57-4a7da3c6d68f/a0ec00c8-1016-421a-a89c-2f1904f8a9f7"
 					(reference "Q2")
@@
 			)
 		)
-		(property "Footprint" "Resistor_SMD:R_0805_2012Metric_Pad1.20x1.40mm_HandSolder"
+		(property "Footprint" "Resistor_SMD:R_0805_2012Metric"
 			(at 142.748 57.15 90)
 			(effects
@@
 		(dnp no)
 		(fields_autoplaced yes)
-		(property "Reference" "#PWR028"
+		(property "Reference" "#PWR032"
 			(at 129.54 83.82 0)
 			(effects
@@
 			(project "nano-m7"
 				(path "/657b92bb-29fd-4612-8c57-4a7da3c6d68f/a0ec00c8-1016-421a-a89c-2f1904f8a9f7"
-					(reference "#PWR028")
-					(unit 1)
-				)
-				(path "/657b92bb-29fd-4612-8c57-4a7da3c6d68f/f2ca9a7d-fea9-4a68-835b-845e026c6569"
-					(reference "#PWR030")
-					(unit 1)
-				)
+					(reference "#PWR032")
+					(unit 1)
+				)
+				(path "/657b92bb-29fd-4612-8c57-4a7da3c6d68f/f2ca9a7d-fea9-4a68-835b-845e026c6569"
+					(reference "#PWR034")
+					(unit 1)
+				)
